Commit message: feat: add lidar sensor and update robot mass properties in URDF files

File: src/my_bot/urdf/gazebo_control.xacro (robot description, xacro)
@@ -27,6 +27,6 @@
     <gazebo reference="caster_wheel">
         <material>Gazebo/Orange</material>
-        <mu1 value="0.001"/>
-        <mu2 value="0.001"/>
+        <mu1 value="0.0001"/>
+        <mu2 value="0.0001"/>
     </gazebo>
 </robot>

File: src/my_bot/urdf/robot.urdf.xacro (robot description, xacro)
@@ -3,3 +3,4 @@
 	<xacro:include filename="robot_core.xacro" />
 	<xacro:include filename="gazebo_control.xacro" />
+	<xacro:include filename="lidar.xacro" />
 </robot>

File: src/my_bot/urdf/robot_core.xacro (robot description, xacro)
@@ -32,5 +32,5 @@
         </collision>
         <inertial>
-            <mass value="0.5"/>
+            <mass value="2.0"/>
             <inertia ixx="0.01" ixy="0.0" ixz="0.0" iyy="0.01" iyz="0.0" izz="0.01"/>
         </inertial>
@@ -100,5 +100,5 @@
         </collision>
         <inertial>
-            <mass value="0.1"/>
+            <mass value="0.01"/>
             <inertia ixx="0.001" ixy="0" ixz="0" iyy="0.001" iyz="0" izz="0.001"/>
         </inertial>

Commit message: fix: Update robot dynamics for smooth control

File: src/my_bot/urdf/gazebo_control.xacro (robot description, xacro)
@@ -7,6 +7,6 @@
             <wheel_separation>0.35</wheel_separation>
             <wheel_diameter>0.1</wheel_diameter>
-            <max_wheel_torque>200</max_wheel_torque>
-            <max_wheel_acceleration>10.0</max_wheel_acceleration>
+            <max_wheel_torque>20</max_wheel_torque>
+            <max_wheel_acceleration>1.0</max_wheel_acceleration>
             <odometry_frame>odom</odometry_frame>
             <robot_base_frame>base_link</robot_base_frame>
@@ -27,6 +27,6 @@
     <gazebo reference="caster_wheel">
         <material>Gazebo/Orange</material>
-        <mu1 value="0.0001"/>
-        <mu2 value="0.0001"/>
+        <mu1 value="0.001"/>
+        <mu2 value="0.001"/>
     </gazebo>
 </robot>

File: src/my_bot/urdf/robot_core.xacro (robot description, xacro)
@@ -32,6 +32,6 @@
         </collision>
         <inertial>
-            <mass value="2.0"/>
-            <inertia ixx="0.01" ixy="0.0" ixz="0.0" iyy="0.01" iyz="0.0" izz="0.01"/>
+            <origin xyz="0.15 0 0.075" rpy="0 0 0"/> <mass value="0.5"/>
+            <inertia ixx="0.003" ixy="0.0" ixz="0.0" iyy="0.003" iyz="0.0" izz="0.003"/>
         </inertial>
     </link>
