Commit message: Use TurtleBot3 Waffle Pi meshes for a more realistic robot model
Replace the primitive box/cylinder robot with the ROBOTIS TurtleBot3
Waffle Pi visual meshes (Apache-2.0) and its real dimensions:
wheel radius 0.033 m, wheel separation 0.288 m, rear ball casters,
LDS lidar on top and the Pi camera at the front face.

All link, joint and frame names (base_link, chassis, left/right_wheel,
laser_frame, camera_link_optical) and sensor/plugin settings are kept,
so SLAM, Nav2 and the behavior nodes need no changes.

- Vendor meshes under src/my_bot/meshes and install them via setup.py
- Export the package share path to GAZEBO_MODEL_PATH so Gazebo can
  resolve package://my_bot/meshes/...
- Update diff_drive geometry and wheel contact parameters
- Add tests for mesh file presence and wheel separation consistency

Co-Authored-By: Claude Opus 5.5 <noreply@anthropic.com>
Claude-Session: https://claude.ai/code/session_01UvGKQAp6qzXeCUvzr9dXXQ

File: src/my_bot/urdf/camera.xacro (robot description, xacro)
@@ -16,13 +16,8 @@
         <parent link="chassis"/>
         <child link="camera_link"/>
-        <origin xyz="0.305 0 0.08" rpy="0 0 0"/>
+        <origin xyz="0.140 0 0.093" rpy="0 0 0"/>
     </joint>
+    <!-- Raspberry Pi camera; its housing is part of the Waffle Pi base mesh -->
     <link name="camera_link">
-        <visual>
-            <geometry>
-                <box size="0.010 0.03 0.03"/>
-            </geometry>
-            <material name="red"/>
-        </visual>
     </link>
     <joint name="camera_optical_joint" type="fixed">
@@ -33,5 +28,4 @@
     <link name="camera_link_optical"></link>
     <gazebo reference="camera_link">
-        <material>Gazebo/Red</material>
         <sensor name="camera" type="camera">
             <pose> 0 0 0 0 0 0 </pose>

File: src/my_bot/urdf/gazebo_control.xacro (robot description, xacro)
@@ -18,6 +18,6 @@
             <left_joint>left_wheel_joint</left_joint>
             <right_joint>right_wheel_joint</right_joint>
-            <wheel_separation>0.35</wheel_separation>
-            <wheel_diameter>0.1</wheel_diameter>
+            <wheel_separation>0.288</wheel_separation>
+            <wheel_diameter>0.066</wheel_diameter>
             <!-- Wheel Dynamics -->
             <max_wheel_torque>20</max_wheel_torque>
@@ -38,26 +38,25 @@
     </gazebo>
     <gazebo reference="chassis">
-        <material>Gazebo/White</material>
+        <material>Gazebo/DarkGrey</material>
     </gazebo>
     <gazebo reference="left_wheel">
-        <material>Gazebo/Blue</material>
+        <material>Gazebo/FlatBlack</material>
         <mu1 value="1.0"/>
         <mu2 value="1.0"/>
-        <kp value="10000000.0"/>
-        <kd value="1.0"/>
+        <kp value="500000.0"/>
+        <kd value="10.0"/>
+        <minDepth>0.001</minDepth>
+        <maxVel>0.1</maxVel>
         <fdir1>1 0 0</fdir1>
     </gazebo>
     <gazebo reference="right_wheel">
-        <material>Gazebo/Blue</material>
+        <material>Gazebo/FlatBlack</material>
         <mu1 value="1.0"/>
         <mu2 value="1.0"/>
-        <kp value="10000000.0"/>
-        <kd value="1.0"/>
+        <kp value="500000.0"/>
+        <kd value="10.0"/>
+        <minDepth>0.001</minDepth>
+        <maxVel>0.1</maxVel>
         <fdir1>1 0 0</fdir1>
     </gazebo>
-    <gazebo reference="caster_wheel">
-        <material>Gazebo/Orange</material>
-        <mu1 value="0.001"/>
-        <mu2 value="0.001"/>
-    </gazebo>
 </robot>

File: src/my_bot/urdf/lidar.xacro (robot description, xacro)
@@ -16,25 +16,26 @@
         <parent link="chassis"/>
         <child link="laser_frame"/>
-        <origin xyz="0.1 0 0.175" rpy="0 0 0"/>
+        <origin xyz="0 0 0.122" rpy="0 0 0"/>
     </joint>
     <link name="laser_frame">
         <visual>
             <geometry>
-                <cylinder radius="0.05" length="0.04"/>
+                <mesh filename="package://my_bot/meshes/lds.stl" scale="0.001 0.001 0.001"/>
             </geometry>
-            <material name="orange"/>
+            <material name="black"/>
         </visual>
         <collision>
+            <origin xyz="0.015 0 -0.0065"/>
             <geometry>
-                <cylinder radius="0.05" length="0.04"/>
+                <cylinder radius="0.055" length="0.0315"/>
             </geometry>
         </collision>
         <inertial>
-            <mass value="0.1"/>
+            <mass value="0.114"/>
             <inertia ixx="0.001" ixy="0" ixz="0" iyy="0.001" iyz="0" izz="0.001"/>
         </inertial>
     </link>
     <gazebo reference="laser_frame">
-        <material>Gazebo/Orange</material>
+        <material>Gazebo/FlatBlack</material>
         <sensor name="laser" type="ray">
             <pose> 0 0 0 0 0 0 </pose>

File: src/my_bot/urdf/robot_core.xacro (robot description, xacro)
@@ -13,37 +13,43 @@
     limitations under the License.
     -->
-    <material name="white">
-        <color rgba="1 1 1 1" />
+    <!--
+    Visual meshes and dimensions follow the ROBOTIS TurtleBot3 Waffle Pi
+    (https://github.com/ROBOTIS-GIT/turtlebot3, Apache-2.0). Link and joint
+    names are kept from the original model so the rest of the stack
+    (diff drive, SLAM, Nav2, behavior nodes) is unaffected.
+    -->
+    <material name="dark_grey">
+        <color rgba="0.25 0.25 0.25 1"/>
     </material>
-    <material name="orange">
-        <color rgba="1 0.3 0.1 1"/>
+    <material name="black">
+        <color rgba="0.1 0.1 0.1 1"/>
     </material>
-    <material name="blue">
-        <color rgba="0.2 0.2 1 1"/>
-    </material>
+    <!-- base_link sits between the drive wheels, 10 mm above the ground -->
     <link name="base_link">
     </link>
+    <!-- chassis origin is the geometric centre of the Waffle Pi body -->
     <joint name="chassis_joint" type="fixed">
         <parent link="base_link"/>
         <child link="chassis"/>
-        <origin xyz="-0.1 0 0"/>
+        <origin xyz="-0.064 0 0"/>
     </joint>
     <link name="chassis">
         <visual>
-            <origin xyz="0.15 0 0.075"/>
             <geometry>
-                <box size="0.3 0.3 0.15"/>
+                <mesh filename="package://my_bot/meshes/waffle_pi_base.stl" scale="0.001 0.001 0.001"/>
             </geometry>
-            <material name="white"/>
+            <material name="dark_grey"/>
         </visual>
         <collision>
-            <origin xyz="0.15 0 0.075"/>
+            <origin xyz="0 0 0.047"/>
             <geometry>
-                <box size="0.3 0.3 0.15"/>
+                <box size="0.266 0.266 0.094"/>
             </geometry>
         </collision>
         <inertial>
-            <origin xyz="0.15 0 0.075" rpy="0 0 0"/> <mass value="0.5"/>
-            <inertia ixx="0.003" ixy="0.0" ixz="0.0" iyy="0.003" iyz="0.0" izz="0.003"/>
+            <origin xyz="0.064 0 0" rpy="0 0 0"/>
+            <mass value="1.3729096"/>
+            <inertia ixx="8.7002718e-03" ixy="-4.7576583e-05" ixz="1.1160499e-04"
+                     iyy="8.6195418e-03" iyz="-3.5422299e-06" izz="1.4612727e-02"/>
         </inertial>
     </link>
@@ -51,22 +57,23 @@
         <parent link="base_link"/>
         <child link="left_wheel"/>
-        <origin xyz="0 0.175 0" rpy="-${pi/2} 0 0" />
+        <origin xyz="0 0.144 0.023" rpy="-${pi/2} 0 0" />
         <axis xyz="0 0 1"/>
     </joint>
     <link name="left_wheel">
         <visual>
+            <origin xyz="0 0 0" rpy="${pi/2} 0 0"/>
             <geometry>
-                <cylinder radius="0.05" length="0.04"/>
+                <mesh filename="package://my_bot/meshes/left_tire.stl" scale="0.001 0.001 0.001"/>
             </geometry>
-            <material name="blue"/>
+            <material name="black"/>
         </visual>
         <collision>
             <geometry>
-                <cylinder radius="0.05" length="0.04"/>
+                <cylinder radius="0.033" length="0.018"/>
             </geometry>
         </collision>
         <inertial>
-            <mass value="0.1"/>
-            <inertia ixx="0.001" ixy="0" ixz="0" iyy="0.001" iyz="0" izz="0.001"/>
+            <mass value="0.028498940"/>
+            <inertia ixx="1.1175580e-05" ixy="0" ixz="0" iyy="1.1192413e-05" iyz="0" izz="2.0712558e-05"/>
         </inertial>
     </link>
@@ -74,45 +81,49 @@
         <parent link="base_link"/>
         <child link="right_wheel"/>
-        <origin xyz="0 -0.175 0" rpy="${pi/2} 0 0" />
-        <axis xyz="0 0 -1"/>
+        <origin xyz="0 -0.144 0.023" rpy="-${pi/2} 0 0" />
+        <axis xyz="0 0 1"/>
     </joint>
     <link name="right_wheel">
         <visual>
+            <origin xyz="0 0 0" rpy="${pi/2} 0 0"/>
             <geometry>
-                <cylinder radius="0.05" length="0.04"/>
+                <mesh filename="package://my_bot/meshes/right_tire.stl" scale="0.001 0.001 0.001"/>
             </geometry>
-            <material name="blue"/>
+            <material name="black"/>
         </visual>
         <collision>
             <geometry>
-                <cylinder radius="0.05" length="0.04"/>
+                <cylinder radius="0.033" length="0.018"/>
             </geometry>
         </collision>
         <inertial>
-            <mass value="0.1"/>
-            <inertia ixx="0.001" ixy="0" ixz="0" iyy="0.001" iyz="0" izz="0.001"/>
+            <mass value="0.028498940"/>
+            <inertia ixx="1.1175580e-05" ixy="0" ixz="0" iyy="1.1192413e-05" iyz="0" izz="2.0712558e-05"/>
         </inertial>
     </link>
-    <joint name="caster_wheel_joint" type="fixed">
-        <parent link="chassis"/>
-        <child link="caster_wheel"/>
-        <origin xyz="0.24 0 0"/>
-    </joint>
-    <link name="caster_wheel">
-        <visual>
-            <geometry>
-                <sphere radius="0.05"/>
-            </geometry>
-            <material name="orange"/>
-        </visual>
-        <collision>
-            <geometry>
-                <sphere radius="0.05"/>
-            </geometry>
-        </collision>
-        <inertial>
-            <mass value="0.01"/>
-            <inertia ixx="0.001" ixy="0" ixz="0" iyy="0.001" iyz="0" izz="0.001"/>
-        </inertial>
-    </link>
+    <!-- Two rear ball casters (their shells are part of the base mesh) -->
+    <xacro:macro name="caster" params="side y">
+        <joint name="caster_${side}_joint" type="fixed">
+            <parent link="chassis"/>
+            <child link="caster_${side}"/>
+            <origin xyz="-0.113 ${y} -0.005"/>
+        </joint>
+        <link name="caster_${side}">
+            <collision>
+                <geometry>
+                    <sphere radius="0.005"/>
+                </geometry>
+            </collision>
+            <inertial>
+                <mass value="0.005"/>
+                <inertia ixx="1e-06" ixy="0" ixz="0" iyy="1e-06" iyz="0" izz="1e-06"/>
+            </inertial>
+        </link>
+        <gazebo reference="caster_${side}">
+            <mu1 value="0.001"/>
+            <mu2 value="0.001"/>
+        </gazebo>
+    </xacro:macro>
+    <xacro:caster side="back_left" y="0.064"/>
+    <xacro:caster side="back_right" y="-0.064"/>
 </robot>
