Commit message: Use a cylinder for the chassis collision to stop lidar ghost hits
The scan showed the chassis outline at 0.12-0.2 m in the front half of
the robot, flickering every frame. Reproduced in gzserver 11 on an empty
ground plane: Gazebo's ODE ray-box test reports hits on a box just below
the scan plane whenever the robot is tilted even slightly, and the robot
rests at ~0.3 deg pitch on its wheels and casters. A static, perfectly
level model gets no hits; the same model at 0.0057 rad gets ~80 per scan.
The old 0.3 m min range started the rays outside the box, which is why
this only appeared after lowering it to 0.12 m.

Raising the lidar or shortening the box only narrows the sector, and
corner boxes bring it back. A cylinder (r = 0.133 m, the body half-width)
gives zero ghost hits at rest and under pitch/roll, and a wall 6 cm from
the bumper is still seen at the right range. The square corners are no
longer in the collision model; Nav2's footprint is unchanged.

Co-Authored-By: Claude Opus 5.5 <noreply@anthropic.com>
Claude-Session: https://claude.ai/code/session_017k5HEXTDq5YPPG2Rsiw6En

File: src/my_bot/urdf/robot_core.xacro (robot description, xacro)
@@ -41,8 +41,13 @@
             <material name="dark_grey"/>
         </visual>
+        <!-- A cylinder, not the 0.266 m box of the real base: Gazebo's ODE
+             ray-box test returns ghost hits on a box just below the scan
+             plane whenever the robot is tilted even slightly (it rests at
+             ~0.3 deg on its casters), so the lidar "saw" the box outline at
+             0.12-0.2 m. Ray-cylinder has no such problem. -->
         <collision>
             <origin xyz="0 0 0.047"/>
             <geometry>
-                <box size="0.266 0.266 0.094"/>
+                <cylinder radius="0.133" length="0.094"/>
             </geometry>
         </collision>
